File: pcb/eagle/OLM-base_v0.2.brd (EAGLE design)
At the start: 45.4 x 63.5 mm, 20 parts, among them IC1 ATMEGA, IC2 MCP1702-33, X1 16 MHz, X2 POWERSUPPLY_DC21MMX

Commit message: added images
Parts:
- moved LED1 7.62 mm to (20.3, 17.8)
- moved X2 7.62 mm to (29.2, 19.1)
- moved X1 2.84 mm to (14.0, 24.1)
Changed lines of the file:
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@@
 <element name="SV1" library="JeeLabs" package="MA04-2" value="SPI/ISP" x="2.54" y="50.8" rot="R270"/>
 <element name="JP1" library="SparkFun" package="1X02_LOCK_LONGPADS" value="BATT" x="6.35" y="19.05" rot="R270"/>
-<element name="X1" library="SparkFun" package="RESONATOR-PTH" value="16 MHz" x="12.7" y="26.67" rot="R270"/>
+<element name="X1" library="SparkFun" package="RESONATOR-PTH" value="16 MHz" x="13.97" y="24.13" rot="R270"/>
 <element name="CON2" library="con-harting" package="CON10L" value="" x="40.64" y="67.31" rot="R270">
 <attribute name="OC_NEWARK" value="unknown" x="-1.27" y="44.45" size="1.778" layer="27" rot="R270" display="off"/>
@@
 <attribute name="OC_FARNELL" value="unknown" x="-1.27" y="44.45" size="1.778" layer="27" rot="R270" display="off"/>
 </element>
-<element name="X2" library="SmartPrj" package="POWERSUPPLY_DC-21MM" value="POWERSUPPLY_DC21MMX" x="21.59" y="19.05" rot="R180"/>
+<element name="X2" library="SmartPrj" package="POWERSUPPLY_DC-21MM" value="POWERSUPPLY_DC21MMX" x="29.21" y="19.05" rot="R180"/>
 <element name="R2" library="resistor" package="0204/7" value="1k" x="11.43" y="36.83" rot="R90"/>
-<element name="LED1" library="eagle-ltspice" package="LED_LD260" value="" x="12.7" y="17.78">
-<attribute name="SPICEMODEL" value="NONE" x="67.31" y="-63.5" size="1.778" layer="27" display="off"/>
-<attribute name="SPICETYPE" value="diode" x="67.31" y="-63.5" size="1.778" layer="27" display="off"/>
-<attribute name="SPICEPREFIX" value="D" x="67.31" y="-63.5" size="1.778" layer="27" display="off"/>
+<element name="LED1" library="eagle-ltspice" package="LED_LD260" value="" x="20.32" y="17.78">
+<attribute name="SPICEMODEL" value="NONE" x="74.93" y="-63.5" size="1.778" layer="27" display="off"/>
+<attribute name="SPICETYPE" value="diode" x="74.93" y="-63.5" size="1.778" layer="27" display="off"/>
+<attribute name="SPICEPREFIX" value="D" x="74.93" y="-63.5" size="1.778" layer="27" display="off"/>
 </element>
 <element name="JP2" library="pinhead" package="2X05" value="" x="40.64" y="49.53" rot="R270"/>
@@
 <wire x1="30.48" y1="33.02" x2="31.75" y2="44.45" width="0" layer="19" extent="1-1"/>
 <wire x1="40.64" y1="26.67" x2="30.48" y2="33.02" width="0" layer="19" extent="1-1"/>
-<wire x1="26.67" y1="22.4028" x2="40.64" y2="26.67" width="0" layer="19" extent="1-1"/>
-<wire x1="21.6662" y1="19.4056" x2="26.67" y2="22.4028" width="0" layer="19" extent="1-1"/>
+<wire x1="34.29" y1="22.4028" x2="40.64" y2="26.67" width="0" layer="19" extent="1-1"/>
+<wire x1="29.2862" y1="19.4056" x2="34.29" y2="22.4028" width="0" layer="19" extent="1-1"/>
 <wire x1="3.81" y1="67.31" x2="11.43" y2="56.261" width="0" layer="19" extent="1-1"/>
 <wire x1="21.59" y1="72.39" x2="31.75" y2="62.23" width="0" layer="19" extent="1-1"/>
 <wire x1="3.81" y1="33.02" x2="3.81" y2="49.53" width="0" layer="19" extent="1-1"/>
-<wire x1="12.7" y1="26.67" x2="3.81" y2="33.02" width="0" layer="19" extent="1-1"/>
-<wire x1="6.35" y1="16.383" x2="12.7" y2="26.67" width="0" layer="19" extent="1-1"/>
+<wire x1="13.97" y1="24.13" x2="3.81" y2="33.02" width="0" layer="19" extent="1-1"/>
+<wire x1="6.35" y1="16.383" x2="13.97" y2="24.13" width="0" layer="19" extent="1-1"/>
 </signal>
 <signal name="N$19">
@@
 <contactref element="IC1" pad="9"/>
 <contactref element="X1" pad="1"/>
-<wire x1="12.7" y1="29.21" x2="17.78" y2="43.18" width="0" layer="19" extent="1-1"/>
+<wire x1="13.97" y1="26.67" x2="17.78" y2="43.18" width="0" layer="19" extent="1-1"/>
 </signal>
 <signal name="N$21">
 <contactref element="IC1" pad="10"/>
 <contactref element="X1" pad="3"/>
-<wire x1="12.7" y1="24.13" x2="17.78" y2="40.64" width="0" layer="19" extent="1-1"/>
+<wire x1="13.97" y1="21.59" x2="17.78" y2="40.64" width="0" layer="19" extent="1-1"/>
 </signal>
 <signal name="VCC" class="1">
@@
 <wire x1="31.75" y1="34.925" x2="31.75" y2="54.61" width="0" layer="19" extent="1-1"/>
 <wire x1="40.64" y1="31.75" x2="31.75" y2="34.925" width="0" layer="19" extent="1-1"/>
-<wire x1="21.6662" y1="25.4" x2="31.75" y2="34.925" width="0" layer="19" extent="1-1"/>
-<wire x1="6.35" y1="19.177" x2="21.6662" y2="25.4" width="0" layer="19" extent="1-1"/>
+<wire x1="29.2862" y1="25.4" x2="31.75" y2="34.925" width="0" layer="19" extent="1-1"/>
+<wire x1="6.35" y1="19.177" x2="29.2862" y2="25.4" width="0" layer="19" extent="1-1"/>
 </signal>
 <signal name="A1">
@@
 <contactref element="R2" pad="1"/>
 <contactref element="LED1" pad="A"/>
-<wire x1="11.43" y1="33.02" x2="11.43" y2="17.78" width="0" layer="19" extent="1-1"/>
+<wire x1="11.43" y1="33.02" x2="19.05" y2="17.78" width="0" layer="19" extent="1-1"/>
 </signal>
 <signal name="RXD">
