File: pcb/eagle/OLM-periph-probe+ambientREVA.brd (EAGLE design)
At the start: 40.6 x 26.7 mm, 6 parts, among them J1 1X2-3.5MM, U2 AM2302

Commit message: fixed terminal
Parts:
- moved J1 1.27 mm to (36.8, 21.6), turned to 90 degrees
Changed lines of the file:
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@@
 <attribute name="OC_FARNELL" value="unknown" x="41.91" y="31.75" size="1.778" layer="27" rot="R90" display="off"/>
 </element>
-<element name="J1" library="adafruit" package="1X2-3.5MM" value="1X2-3.5MM" x="36.83" y="22.86" rot="R270"/>
+<element name="J1" library="adafruit" package="1X2-3.5MM" value="1X2-3.5MM" x="36.83" y="21.59" rot="R90"/>
 <element name="R2" library="resistor" package="0204/7" value="5k" x="5.08" y="20.32"/>
 </elements>
@@
 <contactref element="C2" pad="2"/>
 <wire x1="5.08" y1="8.89" x2="10.33" y2="5.08" width="0" layer="19" extent="1-1"/>
-<wire x1="36.83" y1="24.56" x2="5.08" y2="8.89" width="0" layer="19" extent="1-1"/>
-<wire x1="15.24" y1="19.05" x2="36.83" y2="24.56" width="0" layer="19" extent="1-1"/>
+<wire x1="36.83" y1="19.89" x2="5.08" y2="8.89" width="0" layer="19" extent="1-1"/>
+<wire x1="15.24" y1="19.05" x2="36.83" y2="19.89" width="0" layer="19" extent="1-1"/>
 </signal>
 <signal name="SCK/D13">
@@
 <contactref element="R2" pad="1"/>
 <contactref element="J1" pad="1"/>
-<wire x1="36.83" y1="21.06" x2="1.27" y2="20.32" width="0" layer="19" extent="1-1"/>
-<wire x1="5.08" y1="11.43" x2="36.83" y2="21.06" width="0" layer="19" extent="1-1"/>
+<wire x1="36.83" y1="23.39" x2="1.27" y2="20.32" width="0" layer="19" extent="1-1"/>
+<wire x1="5.08" y1="11.43" x2="36.83" y2="23.39" width="0" layer="19" extent="1-1"/>
 </signal>
 <signal name="SDA/A4">

Commit message: fixed terminal
Parts:
- R1: value 5k -> 10k
- R2: value 5k -> 3k
- moved C2 8.92 mm to (5.08, 19.8)
- moved R2 2.54 mm to (5.08, 22.9)
- moved J1 1.27 mm to (36.8, 22.9)
- moved R1 1.27 mm to (5.08, 25.4)
Changed lines of the file:
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@@
 <setting verticaltext="up"/>
 </settings>
-<grid distance="0.05" unitdist="inch" unit="inch" style="lines" multiple="1" display="no" altdistance="0.025" altunitdist="inch" altunit="inch"/>
+<grid distance="0.01" unitdist="inch" unit="inch" style="lines" multiple="1" display="no" altdistance="0.025" altunitdist="inch" altunit="inch"/>
 <layers>
 <layer number="1" name="Top" color="4" fill="1" visible="yes" active="yes"/>
@@
 <layer number="25" name="tNames" color="7" fill="1" visible="yes" active="yes"/>
 <layer number="26" name="bNames" color="7" fill="1" visible="yes" active="yes"/>
-<layer number="27" name="tValues" color="7" fill="1" visible="yes" active="yes"/>
-<layer number="28" name="bValues" color="7" fill="1" visible="yes" active="yes"/>
+<layer number="27" name="tValues" color="7" fill="1" visible="no" active="yes"/>
+<layer number="28" name="bValues" color="7" fill="1" visible="no" active="yes"/>
 <layer number="29" name="tStop" color="7" fill="3" visible="no" active="yes"/>
 <layer number="30" name="bStop" color="7" fill="6" visible="no" active="yes"/>
@@
 <elements>
 <element name="U2" library="sensor" package="AM2302" value="AM2302" x="24.13" y="8.89" rot="R270"/>
-<element name="C2" library="resistor" package="C025-024X044" value="100n" x="13.97" y="19.05"/>
-<element name="R1" library="resistor" package="0204/7" value="5k" x="5.08" y="24.13"/>
+<element name="C2" library="resistor" package="C025-024X044" value="100n" x="5.08" y="19.812" smashed="yes">
+<attribute name="NAME" x="1.905" y="18.796" size="1.27" layer="25" ratio="10" rot="R90"/>
+<attribute name="VALUE" x="8.382" y="18.415" size="1.27" layer="27" ratio="10"/>
+</element>
+<element name="R1" library="resistor" package="0204/7" value="10k" x="5.08" y="25.4"/>
 <element name="CON1" library="con-harting" package="CON10L" value="" x="3.81" y="8.89" rot="R90">
 <attribute name="OC_NEWARK" value="unknown" x="41.91" y="31.75" size="1.778" layer="27" rot="R90" display="off"/>
@@
 <attribute name="OC_FARNELL" value="unknown" x="41.91" y="31.75" size="1.778" layer="27" rot="R90" display="off"/>
 </element>
-<element name="J1" library="adafruit" package="1X2-3.5MM" value="1X2-3.5MM" x="36.83" y="21.59" rot="R90"/>
-<element name="R2" library="resistor" package="0204/7" value="5k" x="5.08" y="20.32"/>
+<element name="J1" library="adafruit" package="1X2-3.5MM" value="1X2-3.5MM" x="36.83" y="22.86" rot="R90"/>
+<element name="R2" library="resistor" package="0204/7" value="3k" x="5.08" y="22.86"/>
 </elements>
 <signals>
@@
 <contactref element="C2" pad="2"/>
 <wire x1="5.08" y1="8.89" x2="10.33" y2="5.08" width="0" layer="19" extent="1-1"/>
-<wire x1="36.83" y1="19.89" x2="5.08" y2="8.89" width="0" layer="19" extent="1-1"/>
-<wire x1="15.24" y1="19.05" x2="36.83" y2="19.89" width="0" layer="19" extent="1-1"/>
+<wire x1="36.83" y1="21.16" x2="5.08" y2="8.89" width="0" layer="19" extent="1-1"/>
+<wire x1="6.35" y1="19.812" x2="36.83" y2="21.16" width="0" layer="19" extent="1-1"/>
 </signal>
 <signal name="SCK/D13">
@@
 <contactref element="U2" pad="P$2"/>
 <contactref element="R1" pad="1"/>
-<wire x1="5.08" y1="6.35" x2="1.27" y2="24.13" width="0" layer="19" extent="1-1"/>
+<wire x1="5.08" y1="6.35" x2="1.27" y2="25.4" width="0" layer="19" extent="1-1"/>
 <wire x1="10.33" y1="10.16" x2="5.08" y2="6.35" width="0" layer="19" extent="1-1"/>
 </signal>
@@
 <contactref element="R2" pad="1"/>
 <contactref element="J1" pad="1"/>
-<wire x1="36.83" y1="23.39" x2="1.27" y2="20.32" width="0" layer="19" extent="1-1"/>
-<wire x1="5.08" y1="11.43" x2="36.83" y2="23.39" width="0" layer="19" extent="1-1"/>
+<wire x1="36.83" y1="24.66" x2="1.27" y2="22.86" width="0" layer="19" extent="1-1"/>
+<wire x1="5.08" y1="11.43" x2="36.83" y2="24.66" width="0" layer="19" extent="1-1"/>
 </signal>
 <signal name="SDA/A4">
@@
 <contactref element="R2" pad="2"/>
 <contactref element="C2" pad="1"/>
-<wire x1="8.89" y1="20.32" x2="8.89" y2="24.13" width="0" layer="19" extent="1-1"/>
-<wire x1="5.08" y1="3.81" x2="8.89" y2="20.32" width="0" layer="19" extent="1-1"/>
-<wire x1="12.7" y1="19.05" x2="5.08" y2="3.81" width="0" layer="19" extent="1-1"/>
+<wire x1="8.89" y1="22.86" x2="8.89" y2="25.4" width="0" layer="19" extent="1-1"/>
+<wire x1="5.08" y1="3.81" x2="8.89" y2="22.86" width="0" layer="19" extent="1-1"/>
+<wire x1="3.81" y1="19.812" x2="5.08" y2="3.81" width="0" layer="19" extent="1-1"/>
 <wire x1="10.33" y1="12.7" x2="5.08" y2="3.81" width="0" layer="19" extent="1-1"/>
 </signal>
