File: pcb/eagle/OLM-periph-probe+ambientREVA.sch (EAGLE design)
At the start: 6 parts, among them J1 1X2-3.5MM, U2 AM2302

Commit message: fixed terminal
Parts:
- R1: value 5k -> 10k
- R2: value 5k -> 3k
Changed lines of the file:
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@@
 <setting verticaltext="up"/>
 </settings>
-<grid distance="0.05" unitdist="inch" unit="inch" style="lines" multiple="1" display="no" altdistance="0.01" altunitdist="inch" altunit="inch"/>
+<grid distance="0.1" unitdist="inch" unit="inch" style="lines" multiple="1" display="no" altdistance="0.01" altunitdist="inch" altunit="inch"/>
 <layers>
 <layer number="1" name="Top" color="4" fill="1" visible="no" active="no"/>
@@
 <part name="U2" library="sensor" deviceset="AM2302" device="" value="AM2302"/>
 <part name="C2" library="resistor" deviceset="C-EU" device="025-024X044" value="100n"/>
-<part name="R1" library="resistor" deviceset="R-EU_" device="0204/7" value="5k"/>
+<part name="R1" library="resistor" deviceset="R-EU_" device="0204/7" value="10k"/>
 <part name="CON1" library="con-harting" deviceset="CON10L" device=""/>
 <part name="J1" library="adafruit" deviceset="1X2" device="-3.5MM"/>
-<part name="R2" library="resistor" deviceset="R-EU_" device="0204/7" value="5k"/>
+<part name="R2" library="resistor" deviceset="R-EU_" device="0204/7" value="3k"/>
 </parts>
 <sheets>
